File: fan.kicad_sch (KiCad schematic)
At the start: 15 parts, among them J1 Conn_01x04, J2 Conn_01x04_MountingPin, U8 EMC2101

Commit message: update other sheets
Parts:
- C34: renamed from C29; footprint (none) -> Capacitor_SMD:C_0603_1608Metric
- C35: renamed from C30; footprint (none) -> Capacitor_SMD:C_0603_1608Metric
- C36: renamed from C31; footprint (none) -> Capacitor_SMD:C_0603_1608Metric
- C37: renamed from C32; footprint (none) -> Capacitor_SMD:C_0603_1608Metric
- J6: renamed from J1; footprint (none) -> Connector_PinSocket_2.54mm:PinSocket_1x04_P2.54mm_Vertical
- J7: renamed from J2; footprint Connector_PCBEdge:M.2_2280-xx-M -> Connector_JST:JST_SH_BM04B-SRSS-TB_1x04-1MP_P1.00mm_Vertical
- R5: renamed from R4; footprint (none) -> Resistor_SMD:R_0603_1608Metric
- R6: renamed from R5; footprint (none) -> Resistor_SMD:R_0603_1608Metric
- R7: renamed from R6; footprint (none) -> Resistor_SMD:R_0603_1608Metric
- R8: renamed from R7; footprint (none) -> Resistor_SMD:R_0603_1608Metric
- renumbered TP16 to TP25, TP17 to TP26, TP18 to TP27, TP19 to TP28, U8 to U11
Changed lines of the file:
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@@
 		(dnp no)
 		(fields_autoplaced yes)
-		(property "Reference" "C31"
+		(property "Reference" "C36"
 			(at 127 120.6499 0)
 			(effects
@@
 			)
 		)
-		(property "Footprint" ""
+		(property "Footprint" "Capacitor_SMD:C_0603_1608Metric"
 			(at 124.1552 125.73 0)
 			(effects
@@
 			(project "bitcoinMiner"
 				(path "/0beaeab8-8358-4f2b-8329-8eaccffff109/35ae20d3-7baf-4cb1-9480-fa42254bd9a1"
-					(reference "C31")
+					(reference "C36")
 					(unit 1)
 				)
@@
 		(dnp no)
 		(fields_autoplaced yes)
-		(property "Reference" "#PWR028"
+		(property "Reference" "#PWR027"
 			(at 109.22 133.35 0)
 			(effects
@@
 			(project "bitcoinMiner"
 				(path "/0beaeab8-8358-4f2b-8329-8eaccffff109/35ae20d3-7baf-4cb1-9480-fa42254bd9a1"
-					(reference "#PWR028")
+					(reference "#PWR027")
 					(unit 1)
 				)
@@
 		(dnp no)
 		(fields_autoplaced yes)
-		(property "Reference" "U8"
+		(property "Reference" "U11"
 			(at 151.13 60.96 0)
 			(effects
@@
 			(project "bitcoinMiner"
 				(path "/0beaeab8-8358-4f2b-8329-8eaccffff109/35ae20d3-7baf-4cb1-9480-fa42254bd9a1"
-					(reference "U8")
+					(reference "U11")
 					(unit 1)
 				)
@@
 		(on_board yes)
 		(dnp no)
-		(property "Reference" "R6"
+		(property "Reference" "R7"
 			(at 120.65 106.172 0)
 			(effects
@@
 			)
 		)
-		(property "Footprint" ""
+		(property "Footprint" "Resistor_SMD:R_0603_1608Metric"
 			(at 118.11 107.95 0)
 			(effects
@@
 			(project "bitcoinMiner"
 				(path "/0beaeab8-8358-4f2b-8329-8eaccffff109/35ae20d3-7baf-4cb1-9480-fa42254bd9a1"
-					(reference "R6")
+					(reference "R7")
 					(unit 1)
 				)
@@
 		(dnp no)
 		(fields_autoplaced yes)
-		(property "Reference" "R4"
+		(property "Reference" "R5"
 			(at 110.49 64.77 90)
 			(effects
@@
 			)
 		)
-		(property "Footprint" ""
+		(property "Footprint" "Resistor_SMD:R_0603_1608Metric"
 			(at 110.49 71.12 0)
 			(effects
@@
 			(project "bitcoinMiner"
 				(path "/0beaeab8-8358-4f2b-8329-8eaccffff109/35ae20d3-7baf-4cb1-9480-fa42254bd9a1"
-					(reference "R4")
+					(reference "R5")
 					(unit 1)
 				)
@@
 		(dnp no)
 		(fields_autoplaced yes)
-		(property "Reference" "#PWR027"
+		(property "Reference" "#PWR026"
 			(at 96.52 121.92 0)
 			(effects
@@
 			(project "bitcoinMiner"
 				(path "/0beaeab8-8358-4f2b-8329-8eaccffff109/35ae20d3-7baf-4cb1-9480-fa42254bd9a1"
-					(reference "#PWR027")
+					(reference "#PWR026")
 					(unit 1)
 				)
@@
 		(dnp no)
 		(fields_autoplaced yes)
-		(property "Reference" "#PWR031"
+		(property "Reference" "#PWR030"
 			(at 165.1 86.36 0)
 			(effects
@@
 			(project "bitcoinMiner"
 				(path "/0beaeab8-8358-4f2b-8329-8eaccffff109/35ae20d3-7baf-4cb1-9480-fa42254bd9a1"
-					(reference "#PWR031")
+					(reference "#PWR030")
 					(unit 1)
 				)
@@
 		(on_board yes)
 		(dnp no)
-		(property "Reference" "C32"
+		(property "Reference" "C37"
 			(at 189.23 72.3899 0)
 			(effects
@@
 			)
 		)
-		(property "Footprint" ""
+		(property "Footprint" "Capacitor_SMD:C_0603_1608Metric"
 			(at 186.3852 77.47 0)
 			(effects
@@
 			(project "bitcoinMiner"
 				(path "/0beaeab8-8358-4f2b-8329-8eaccffff109/35ae20d3-7baf-4cb1-9480-fa42254bd9a1"
-					(reference "C32")
+					(reference "C37")
 					(unit 1)
 				)
@@
 		(dnp no)
 		(fields_autoplaced yes)
-		(property "Reference" "J2"
+		(property "Reference" "J7"
 			(at 166.37 115.2143 0)
 			(effects
@@
 			)
 		)
-		(property "Footprint" "Connector_PCBEdge:M.2_2280-xx-M"
+		(property "Footprint" "Connector_JST:JST_SH_BM04B-SRSS-TB_1x04-1MP_P1.00mm_Vertical"
 			(at 163.83 118.11 0)
 			(effects
@@
 			(project "bitcoinMiner"
 				(path "/0beaeab8-8358-4f2b-8329-8eaccffff109/35ae20d3-7baf-4cb1-9480-fa42254bd9a1"
-					(reference "J2")
+					(reference "J7")
 					(unit 1)
 				)
@@
 		(on_board yes)
 		(dnp no)
-		(property "Reference" "C29"
+		(property "Reference" "C34"
 			(at 114.3 120.6499 0)
 			(effects
@@
 			)
 		)
-		(property "Footprint" ""
+		(property "Footprint" "Capacitor_SMD:C_0603_1608Metric"
 			(at 117.1448 125.73 0)
 			(effects
@@
 			(project "bitcoinMiner"
 				(path "/0beaeab8-8358-4f2b-8329-8eaccffff109/35ae20d3-7baf-4cb1-9480-fa42254bd9a1"
-					(reference "C29")
+					(reference "C34")
 					(unit 1)
 				)
@@
 		(dnp no)
 		(fields_autoplaced yes)
-		(property "Reference" "#PWR030"
+		(property "Reference" "#PWR029"
 			(at 135.89 69.85 0)
 			(effects
@@
 			(project "bitcoinMiner"
 				(path "/0beaeab8-8358-4f2b-8329-8eaccffff109/35ae20d3-7baf-4cb1-9480-fa42254bd9a1"
-					(reference "#PWR030")
+					(reference "#PWR029")
 					(unit 1)
 				)
@@
 		(on_board yes)
 		(dnp no)
-		(property "Reference" "TP17"
+		(property "Reference" "TP26"
 			(at 101.6 94.996 90)
 			(effects
@@
 			(project "bitcoinMiner"
 				(path "/0beaeab8-8358-4f2b-8329-8eaccffff109/35ae20d3-7baf-4cb1-9480-fa42254bd9a1"
-					(reference "TP17")
+					(reference "TP26")
 					(unit 1)
 				)
@@
 		(dnp no)
 		(fields_autoplaced yes)
-		(property "Reference" "J1"
+		(property "Reference" "J6"
 			(at 142.24 106.68 0)
 			(effects
@@
 			)
 		)
-		(property "Footprint" ""
+		(property "Footprint" "Connector_PinSocket_2.54mm:PinSocket_1x04_P2.54mm_Vertical"
 			(at 142.24 118.11 0)
 			(effects
@@
 			(project "bitcoinMiner"
 				(path "/0beaeab8-8358-4f2b-8329-8eaccffff109/35ae20d3-7baf-4cb1-9480-fa42254bd9a1"
-					(reference "J1")
+					(reference "J6")
 					(unit 1)
 				)
@@
 		(on_board yes)
 		(dnp no)
-		(property "Reference" "C30"
+		(property "Reference" "C35"
 			(at 115.57 73.6599 0)
 			(effects
@@
 			)
 		)
-		(property "Footprint" ""
+		(property "Footprint" "Capacitor_SMD:C_0603_1608Metric"
 			(at 118.4148 78.74 0)
 			(effects
@@
 			(project "bitcoinMiner"
 				(path "/0beaeab8-8358-4f2b-8329-8eaccffff109/35ae20d3-7baf-4cb1-9480-fa42254bd9a1"
-					(reference "C30")
+					(reference "C35")
 					(unit 1)
 				)
@@
 		(on_board yes)
 		(dnp no)
-		(property "Reference" "TP19"
+		(property "Reference" "TP28"
 			(at 132.08 105.664 0)
 			(effects
@@
 			(project "bitcoinMiner"
 				(path "/0beaeab8-8358-4f2b-8329-8eaccffff109/35ae20d3-7baf-4cb1-9480-fa42254bd9a1"
-					(reference "TP19")
+					(reference "TP28")
 					(unit 1)
 				)
@@
 		(dnp no)
 		(fields_autoplaced yes)
-		(property "Reference" "R7"
+		(property "Reference" "R8"
 			(at 177.8 68.5799 0)
 			(effects
@@
 			)
 		)
-		(property "Footprint" ""
+		(property "Footprint" "Resistor_SMD:R_0603_1608Metric"
 			(at 175.26 69.85 0)
 			(effects
@@
 			(project "bitcoinMiner"
 				(path "/0beaeab8-8358-4f2b-8329-8eaccffff109/35ae20d3-7baf-4cb1-9480-fa42254bd9a1"
-					(reference "R7")
+					(reference "R8")
 					(unit 1)
 				)
@@
 		(dnp no)
 		(fields_autoplaced yes)
-		(property "Reference" "#PWR029"
+		(property "Reference" "#PWR028"
 			(at 118.11 107.95 0)
 			(effects
@@
 			(project "bitcoinMiner"
 				(path "/0beaeab8-8358-4f2b-8329-8eaccffff109/35ae20d3-7baf-4cb1-9480-fa42254bd9a1"
-					(reference "#PWR029")
+					(reference "#PWR028")
 					(unit 1)
 				)
@@
 		(on_board yes)
 		(dnp no)
-		(property "Reference" "R5"
+		(property "Reference" "R6"
 			(at 110.49 85.09 90)
 			(effects
@@
 			)
 		)
-		(property "Footprint" ""
+		(property "Footprint" "Resistor_SMD:R_0603_1608Metric"
 			(at 110.49 78.74 0)
 			(effects
@@
 			(project "bitcoinMiner"
 				(path "/0beaeab8-8358-4f2b-8329-8eaccffff109/35ae20d3-7baf-4cb1-9480-fa42254bd9a1"
-					(reference "R5")
+					(reference "R6")
 					(unit 1)
 				)
@@
 		(dnp no)
 		(fields_autoplaced yes)
-		(property "Reference" "#PWR032"
+		(property "Reference" "#PWR031"
 			(at 180.34 68.58 0)
 			(effects
@@
 			(project "bitcoinMiner"
 				(path "/0beaeab8-8358-4f2b-8329-8eaccffff109/35ae20d3-7baf-4cb1-9480-fa42254bd9a1"
-					(reference "#PWR032")
+					(reference "#PWR031")
 					(unit 1)
 				)
@@
 		(on_board yes)
 		(dnp no)
-		(property "Reference" "TP16"
+		(property "Reference" "TP25"
 			(at 101.6 54.864 90)
 			(effects
@@
 			(project "bitcoinMiner"
 				(path "/0beaeab8-8358-4f2b-8329-8eaccffff109/35ae20d3-7baf-4cb1-9480-fa42254bd9a1"
-					(reference "TP16")
+					(reference "TP25")
 					(unit 1)
 				)
@@
 		(on_board yes)
 		(dnp no)
-		(property "Reference" "TP18"
+		(property "Reference" "TP27"
 			(at 113.03 108.204 0)
 			(effects
@@
 			(project "bitcoinMiner"
 				(path "/0beaeab8-8358-4f2b-8329-8eaccffff109/35ae20d3-7baf-4cb1-9480-fa42254bd9a1"
-					(reference "TP18")
-					(unit 1)
-				)
+					(reference "TP27")
+					(unit 1)
+				)
