File: esp32.kicad_sch (KiCad schematic)
At the start: 21 parts, among them J3 Conn_01x04, J3 TC2030-IDC, J4 Conn_01x06, J5 USB_C_Receptacle_USB2.0, SW1 GT-TC029B-H025-L1N, SW2 GT-TC029B-H025-L1N, U10 RT9080-33GJ5, U11 ESP32-S3-WROOM-1

Commit message: update other sheets
Parts:
- renumbered C53 to C29, C54 to C30, C55 to C31, C56 to C32, C57 to C33, J3 to J2, R23 to R4, TP22 to TP18, TP23 to TP19, TP24 to TP20, TP25 to TP21, TP26 to TP22, TP27 to TP23, TP28 to TP24, U11 to U10, U10 to U9
Connections:
- net RXD0: now reaches U10.12 (GPIO8/TOUCH8/ADC1_CH7/SUBSPICS1)
- net GPIO46: now reaches U10.16 (*GPIO46)
- net RXD1: now reaches U10.17 (GPIO9/TOUCH9/ADC1_CH8/FSPIHD/SUBSPIHD)
- net CRS_DV: now reaches U10.18 (GPIO10/TOUCH10/ADC1_CH9/FSPICS0/FSPIIO4/SUBSPICS0)
- net REF_CLK: now reaches U10.20 (GPIO12/TOUCH12/ADC2_CH1/FSPICLK/FSPIIO6/SUBSPICLK)
- net MDIO: now reaches U10.22 (GPIO14/TOUCH14/ADC2_CH3/FSPIWP/FSPIDQS/SUBSPIWP)
- net GPIO21: now reaches U10.23 (GPIO21)
- net GPIO45: now reaches U10.26 (*GPIO45)
- net GPIO35: now reaches U10.28 (SPIIO6/GPIO35/FSPID/SUBSPID)
- net GPIO36: now reaches U10.29 (SPIIO7/GPIO36/FSPICLK/SUBSPICLK)
- net GPIO37: now reaches U10.30 (SPIDQS/GPIO37/FSPIQ/SUBSPIQ)
- net GPIO38: now reaches U10.31 (GPIO38/FSPIWP/SUBSPIWP)
- net TXD0: now reaches U10.4 (GPIO4/TOUCH4/ADC1_CH3)
- net TXD1: now reaches U10.5 (GPIO5/TOUCH5/ADC1_CH4)
- net TX_EN: now reaches U10.7 (GPIO7/TOUCH7/ADC1_CH6)
- net MDC: now reaches U10.8 (GPIO15/U0RTS/ADC2_CH4/XTAL_32K_P)
- no-connect marks 24 -> 8
Other:
- note added: "Used for Internal Flash ->"
- moved on the sheet: J4, SW2, TP21, U10

Commit message: updates
Parts:
- J3: footprint bitaxe:PinHeader_1x04_P2.54mm_Vertical_shifted -> Connector_PinHeader_2.54mm:PinHeader_1x04_P2.54mm_Vertical
Other:
- moved on the sheet: C30, R4, SW1, U10
