File: power.kicad_sch (KiCad schematic)
At the start: 40 parts, among them T1 net-tie, U9 TPS546D24ARVFR

Commit message: update power sheet
Parts:
- R10: renamed from R9; footprint Resistor_SMD:R_0402_1005Metric -> Resistor_SMD:R_0603_1608Metric
- R11: renamed from R10; footprint Resistor_SMD:R_0402_1005Metric -> Resistor_SMD:R_0603_1608Metric
- R12: renamed from R11; footprint Resistor_SMD:R_0402_1005Metric -> Resistor_SMD:R_0603_1608Metric
- R13: renamed from R12; footprint Resistor_SMD:R_0402_1005Metric -> Resistor_SMD:R_0603_1608Metric
- R14: renamed from R13; footprint Resistor_SMD:R_0402_1005Metric -> Resistor_SMD:R_0603_1608Metric
- R15: renamed from R14; footprint Resistor_SMD:R_0402_1005Metric -> Resistor_SMD:R_0603_1608Metric
- R16: renamed from R15; footprint Resistor_SMD:R_0402_1005Metric -> Resistor_SMD:R_0603_1608Metric
- R17: renamed from R16; footprint Resistor_SMD:R_0402_1005Metric -> Resistor_SMD:R_0603_1608Metric
- R18: renamed from R17; footprint Resistor_SMD:R_0402_1005Metric -> Resistor_SMD:R_0603_1608Metric
- R19: renamed from R18; footprint Resistor_SMD:R_0402_1005Metric -> Resistor_SMD:R_0603_1608Metric
- R21: renamed from R20; footprint Resistor_SMD:R_0402_1005Metric -> Resistor_SMD:R_0603_1608Metric
- R22: renamed from R21; footprint Resistor_SMD:R_0402_1005Metric -> Resistor_SMD:R_0603_1608Metric
- R23: renamed from R22; footprint Resistor_SMD:R_0402_1005Metric -> Resistor_SMD:R_0603_1608Metric
- R9: renamed from R8; footprint Resistor_SMD:R_0402_1005Metric -> Resistor_SMD:R_0603_1608Metric
- renumbered C33 to C38, C34 to C39, C35 to C40, C36 to C41, C37 to C42, C38 to C43, C39 to C44, C40 to C45, C41 to C46, C42 to C47, C43 to C48, C44 to C49, C45 to C50, C46 to C51, C47 to C52, C48 to C53, C49 to C54, C50 to C55, C51 to C56, C52 to C57, R19 to R20, TP20 to TP29, TP21 to TP30, U9 to U12

Commit message: updates
Changed lines of the file:
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@@
-		)
-	)
-	(global_label "VIN"
-		(shape input)
-		(at 49.53 22.86 180)
-		(fields_autoplaced yes)
-		(effects
-			(font
-				(size 1.27 1.27)
-			)
-			(justify right)
-		)
-		(property "Intersheetrefs" "${INTERSHEET_REFS}"
-			(at 43.5209 22.86 0)
-			(effects
-				(font
-					(size 1.27 1.27)
-				)
-				(justify right)
-				(hide yes)
-			)
 		)
 	)
@@
 		(effects
 			(font
+				(size 1.27 1.27)
+			)
+			(justify right)
+		)
+	)
+	(hierarchical_label "VIN"
+		(shape input)
+		(at 49.53 22.86 180)
+		(effects
+			(font
