File: bm1370.kicad_sch (KiCad schematic)
At the start: 53 parts, among them U1 25MHz, U2 MCP1824T-1202E/OT, U3 MCP1824T-0802E, U4 BM1370_mode1, U5 SN74LVC1T45DBV, U6 SN74LVC1T45DBV, U7 SN74LVC1T45DBV

Commit message: update other sheets
Parts:
- C1, C10, C11, C12, C13, C14, C15, C16, C17, C18, C19, C2, C20, C21, C22, C23, C24, C25, C26, C27, C28, C3, C4, C5, C6, C7, C8, C9: footprint (none) -> Capacitor_SMD:C_0603_1608Metric
- R1, R2, R3: footprint (none) -> Resistor_SMD:R_0603_1608Metric
- U2: renamed from U1; footprint (none) -> Crystal:Crystal_SMD_2016-4Pin_2.0x1.6mm
- renumbered TP8 to TP10, TP9 to TP11, TP10 to TP12, TP11 to TP13, TP12 to TP14, TP13 to TP15, TP14 to TP16, TP15 to TP17, TP1 to TP3, TP2 to TP4, TP3 to TP5, TP4 to TP6, TP5 to TP7, TP6 to TP8, TP7 to TP9, U2 to U3, U3 to U4, U4 to U5, U5 to U6, U6 to U7, U7 to U8

Commit message: updates
Connections:
- net VDD: now reaches C13.2, C18.1, U5.31 (VDD)
Changed lines of the file:
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@@
+	)
+	(junction
+		(at 158.75 92.71)
+		(diameter 0)
+		(color 0 0 0 0)
 	)
 	(junction
@@
 	(wire
 		(pts
+			(xy 160.02 90.17) (xy 158.75 90.17)
+		)
+		(stroke
+			(width 0)
+			(type default)
+		)
+	)
+	(wire
+		(pts
 			(xy 142.24 129.54) (xy 143.51 129.54)
 		)
@@
 	(wire
 		(pts
+			(xy 158.75 92.71) (xy 161.29 92.71)
+		)
+		(stroke
+			(width 0)
+			(type default)
+		)
+	)
+	(wire
+		(pts
 			(xy 115.57 41.91) (xy 115.57 43.18)
 		)
@@
 	(wire
 		(pts
-			(xy 143.51 92.71) (xy 161.29 92.71)
+			(xy 143.51 92.71) (xy 158.75 92.71)
 		)
 		(stroke
@@
 		(pts
 			(xy 264.16 46.99) (xy 264.16 49.53)
+		)
+		(stroke
+			(width 0)
+			(type default)
+		)
+	)
+	(wire
+		(pts
+			(xy 158.75 90.17) (xy 158.75 92.71)
 		)
 		(stroke
@@
 		)
 	)
+	(hierarchical_label "VDD"
+		(shape input)
+		(at 160.02 90.17 0)
+		(effects
+			(font
+				(size 1.27 1.27)
+			)
+			(justify left)
+		)
+	)

Commit message: update pcb
Connections:
- net VDD: now also C12.2, C15.2, C16.2, C7.2, C9.2
Changed lines of the file:
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@@
+	(wire
+		(pts
+			(xy 133.35 30.48) (xy 133.35 33.02)
+		)
+		(stroke
+			(width 0)
+			(type default)
+		)
+	)
 	(wire
 		(pts
@@
 		)
 	)
+	(hierarchical_label "VDD"
+		(shape input)
+		(at 133.35 30.48 0)
+		(effects
+			(font
+				(size 1.27 1.27)
+			)
+			(justify left)
+		)
+	)
