File: bitcoinMiner.kicad_pcb (KiCad board)
At the start: 4 copper layers, 80 x 80 mm, 179 parts, among them J1 54-00164, J2 TC2030-IDC, J3 Conn_01x04, J4 Conn_01x06, J5 USB_C_Receptacle_USB2.0, J6 Conn_01x04, J7 Conn_01x04_MountingPin, J8 RJ45_Bel_SI-60062-F, SW1 GT-TC029B-H025-L1N, SW2 GT-TC029B-H025-L1N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

Commit message: updates
Parts:
- J3: footprint bitaxe:PinHeader_1x04_P2.54mm_Vertical_shifted -> Connector_PinHeader_2.54mm:PinHeader_1x04_P2.54mm_Vertical
- moved J3 237.3 mm to (62.4, 30.0), turned to 90 degrees
- moved J4 234.4 mm to (56.4, 30.0), turned to -90 degrees
- moved C29 231.9 mm to (56.5, 42.3), turned to -90 degrees
- moved C31 227.7 mm to (56.5, 50.0), turned to 90 degrees
- moved U9 227.7 mm to (56.5, 46.0), turned to -90 degrees
- moved C28 156.7 mm to (67.3, 37.6), turned to 90 degrees
- moved C24 154.9 mm to (71.2, 42.5), turned to 90 degrees
- moved C27 152.5 mm to (73.0, 37.7), turned to 90 degrees
- moved C23 151.3 mm to (76.8, 42.5), turned to 90 degrees
- moved C26 148.6 mm to (78.5, 37.7), turned to 90 degrees
- moved C3 141.6 mm to (109.0, 38.8)
- moved C25 140.9 mm to (65.8, 42.5), turned to 90 degrees
- moved U2 140.4 mm to (109.0, 35.5)
- moved H5 140.3 mm to (60.0, 37.5)
- moved C37 138.8 mm to (86.8, 38.8), turned to 180 degrees
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Connections:
- C1 pad 1: VIN -> +5V
- C13 pad 2: Net-(U5-VDD) -> /VDD
- C18 pad 1: Net-(U5-VDD) -> /VDD
- C2 pad 1: VIN -> +5V
- C34 pad 1: VIN -> +5V
- C36 pad 1: VIN -> +5V
- C37 pad 1: VIN -> +5V
- C39 pad 1: VIN -> +5V
- C40 pad 1: VIN -> +5V
- C41 pad 1: VIN -> +5V
- C43 pad 1: VIN -> +5V
- C44 pad 1: VIN -> +5V
- C46 pad 1: VIN -> +5V
- J1 pad 1: /VIN -> +5V
- J6 pad 2: VIN -> +5V
- J7 pad 2: VIN -> +5V
- R17 pad 1: VIN -> +5V
- R19 pad 1: VIN -> +5V
- R25 pad 2: /Ethernet/RESET -> /ESP32/GPIO21
- R8 pad 1: VIN -> +5V
- TP1 pad 1: /VIN -> +5V
- U12 pad 21: VIN -> +5V
- U12 pad 22: VIN -> +5V
- U12 pad 23: VIN -> +5V
- U12 pad 24: VIN -> +5V
- U12 pad 25: VIN -> +5V
- U13 pad 15: /Ethernet/AGND -> GND
- U13 pad 19: /Ethernet/AGND -> GND
- U13 pad 29: /Ethernet/RESET -> /ESP32/GPIO21
- U13 pad 7: /Ethernet/PWR_DOWN -> /ESP32/GPIO35
- U3 pad 1: VIN -> +5V
- U3 pad 3: VIN -> +5V
- U4 pad 1: VIN -> +5V
- U4 pad 3: VIN -> +5V
- U5 pad 31: Net-(U5-VDD) -> /VDD
Routing:
- net GND: track 58.0 -> 282.1 mm, vias 17 -> 82
- net /3V3: track 7.31 -> 92.5 mm, vias 2 -> 3
- net +5V: track 0.00 -> 74.9 mm, vias 0 -> 18
- net +3V3: track 0.00 -> 52.0 mm, vias 0 -> 3
- net /ESP32/USB_D+: track 2.44 -> 49.6 mm
- net /ESP32/USB_D-: track 2.44 -> 48.7 mm
- net /ESP32/CRS_DV: track 0.00 -> 37.9 mm, vias 0 -> 2
- net /ESP32/RXD1: track 0.00 -> 35.6 mm, vias 0 -> 2
- net FAN_PWM: track 0.00 -> 35.5 mm
- net +1V2: track 0.00 -> 35.5 mm, vias 0 -> 3
- net /ESP32/TXD0: track 2.30 -> 32.2 mm, vias 1 -> 2
- net /ESP32/TX_EN: track 2.12 -> 29.6 mm, vias 1 -> 2
- net /ESP32/RXD0: track 0.00 -> 27.0 mm, vias 0 -> 2
- net /ESP32/TXD1: track 1.76 -> 28.5 mm, vias 1 -> 2
- net /VDD: track 0.00 -> 25.4 mm, vias 0 -> 14
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- added copper zone on In2.Cu, net +3V3
- added copper zone on F.Cu, net +5V
Other:
- outline, holes or cut-outs redrawn

Commit message: update pcb
Parts:
- C12, C15, C16, C7, C9: moved to B.Cu
- moved FID2 181.9 mm to (27.5, 62.5)
- moved FID1 181.7 mm to (27.5, 82.5)
- moved FID8 155.8 mm to (57.5, 62.5)
- moved FID7 155.4 mm to (57.5, 87.5)
- moved R2 145.5 mm to (61.8, 51.5)
- moved C8 143.7 mm to (73.2, 51.8), turned to -90 degrees
- moved FID3 142.7 mm to (75.0, 30.0)
- moved R3 141.5 mm to (64.8, 57.2), turned to 90 degrees
- moved C16 139.9 mm to (76.5, 55.8), turned to 90 degrees
- moved R1 139.2 mm to (68.0, 53.5)
- moved C6 139.1 mm to (71.5, 51.8), turned to -90 degrees
- moved C22 137.5 mm to (88.5, 51.8), turned to 90 degrees
- moved C15 137.1 mm to (78.2, 55.8), turned to 90 degrees
- moved C13 136.4 mm to (76.8, 51.8), turned to -90 degrees
- moved R23 135.7 mm to (71.0, 89.5), turned to 180 degrees
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Connections:
- C12 pad 2: Net-(C12-Pad2) -> /VDD
- C15 pad 2: Net-(C12-Pad2) -> /VDD
- C16 pad 2: Net-(C12-Pad2) -> /VDD
- C7 pad 2: Net-(C12-Pad2) -> /VDD
- C9 pad 2: Net-(C12-Pad2) -> /VDD
Routing:
- net /ESP32/MDIO: track 5.93 -> 53.1 mm, vias 0 -> 2
- net /ESP32/GPIO21: track 6.74 -> 47.1 mm, vias 0 -> 4
- net /VDD: track 25.4 -> 59.6 mm, vias 14 -> 29
- net +1V2: track 35.5 -> 63.3 mm, vias 3 -> 5
- net +5V: track 74.9 -> 96.3 mm, vias 18 -> 20
- net Net-(U5-LITE_PAD): track 0.00 -> 20.9 mm, vias 0 -> 2
- net CI: track 14.9 -> 35.2 mm, vias 0 -> 2
- net Net-(U5-ROSC_SEL): track 0.00 -> 17.0 mm
- net RST_N: track 16.3 -> 32.5 mm
- net PIN_MODE: track 0.00 -> 15.2 mm, vias 0 -> 2
- net GND: track 282.1 -> 297.0 mm, vias 82 -> 90
- net CLKO: track 0.00 -> 14.0 mm, vias 0 -> 2
- net Net-(U12-BP1V5): track 10.5 -> 24.1 mm, vias 0 -> 2
- net BI: track 0.00 -> 12.9 mm
- net Net-(U12-ADRSEL): track 2.27 -> 14.6 mm, vias 0 -> 4
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- added copper zone on B.Cu, net /VDD

Commit message: update pcb
Parts:
- G***: moved to B.Cu
- moved SW1 268.5 mm to (26.8, 67.8), turned to 90 degrees
- moved C30 263.4 mm to (29.2, 68.8), turned to -90 degrees
- moved R4 263.0 mm to (29.3, 66.8), turned to -90 degrees
- moved SW2 253.2 mm to (26.8, 73.7), turned to -90 degrees
- moved TP21 248.8 mm to (27.0, 59.2)
- moved TP19 246.9 mm to (35.5, 33.8)
- moved TP20 245.0 mm to (39.0, 33.8)
- moved TP24 237.9 mm to (50.0, 34.2)
- moved TP18 235.3 mm to (37.8, 60.2)
- moved TP22 221.0 mm to (57.5, 55.5)
- moved TP23 180.1 mm to (102.8, 54.2), turned to 180 degrees
- moved G*** 87.7 mm to (62.9, 59.8), turned to -90 degrees
- moved R1 0.25 mm to (67.8, 53.5)
Routing:
- net /ESP32/IO0: track 1.39 -> 68.3 mm, vias 1 -> 3
- net /SCL: track 20.6 -> 83.9 mm, vias 0 -> 2
- net /SDA: track 23.7 -> 84.4 mm, vias 0 -> 2
- net /ESP32/GPIO35: track 0.00 -> 56.3 mm, vias 0 -> 6
- net /Power/PGOOD: track 3.09 -> 54.2 mm, vias 2 -> 3
- net /VDD: track 59.6 -> 108.6 mm, vias 29 -> 30
- net +3V3: track 52.0 -> 94.3 mm, vias 4 -> 5
- net +5V: track 96.3 -> 129.9 mm, vias 20 -> 24
- net /ESP32/EN: track 28.1 -> 51.3 mm, vias 2 -> 3
- net /3V3: track 92.5 -> 113.4 mm, vias 3 -> 5
- net +1V2: track 63.3 -> 82.8 mm, vias 5 -> 6
- net GND: track 297.0 -> 301.6 mm, vias 90 -> 91
- net /ESP32/P_TX: track 6.33 -> 9.83 mm
- added copper zone on B.Cu, net GND
