File: kicad/_restore_backup_2026-08-12T20-21-57-306/bitcoinMiner.kicad_pcb (KiCad board)
At the start: 6 copper layers, 75 x 100 mm, 148 parts, among them J1 54-00164, J2 TC2030-IDC, J3 Conn_01x06, J4 USB_C_Receptacle_USB2.0_14P, J5 Conn_01x04, J6 Conn_01x04, J7 Conn_01x04_MountingPin, SW1 SW_Push, SW2 SW_Push, T1 net-tie, U10 ESP32-S3-WROOM-1, U11 EMC2101, U12 TPS546D24ARVFR, U2 25MHz, U3 TLV75712PDBV, U4 MCP1824T-0802E, U5 BM1370_mode1, U6 SN74LVC1T45DBV, U7 SN74LVC1T45DBV, U8 SN74LVC1T45DBV, U9 TLV75733PDBV

Commit message: finish schematic
Parts:
- moved C32 262.0 mm to (265.9, 146.8), turned to 0 degrees
- moved C31 257.9 mm to (272.0, 132.5), turned to -90 degrees
- moved U9 254.1 mm to (269.0, 132.5), turned to 0 degrees
- moved C29 250.3 mm to (266.0, 132.5), turned to -90 degrees
- moved C33 242.5 mm to (262.2, 147.6)
- moved J2 234.8 mm to (242.4, 153.5)
Connections:
- U10 pad 10: TX -> /TX
- U10 pad 11: RX -> /RX
- U10 pad 39: RST -> /RST
Routing:
- net RST: track 44.6 -> 0.00 mm, vias 2 -> 0
- net /VDD: track 39.5 -> 0.00 mm, vias 2 -> 0
- net RX: track 38.5 -> 0.00 mm, vias 2 -> 0
- net TX: track 32.0 -> 0.00 mm, vias 2 -> 0
- net /ESP32/P_RX: track 22.5 -> 0.00 mm, vias 2 -> 0
- net /ESP32/P_TX: track 22.4 -> 0.00 mm, vias 2 -> 0
- net /ESP32/EN: track 60.8 -> 40.7 mm, vias 3 -> 2
- net /3V3: track 15.3 -> 1.90 mm, vias 2 -> 1
- net /ESP32/IO0: track 53.8 -> 43.4 mm, vias 2 -> 0
- net GND: track 38.2 -> 31.3 mm, vias 50 -> 44
- net /5V: track 6.04 -> 0.00 mm
