File: kicad/_restore_backup_2026-08-12T20-21-57-306/esp32.kicad_sch (KiCad schematic)
At the start: 21 parts, among them J2 TC2030-IDC, J3 Conn_01x06, J4 USB_C_Receptacle_USB2.0_14P, J5 Conn_01x04, SW1 SW_Push, SW2 SW_Push, U10 ESP32-S3-WROOM-1, U9 TLV75733PDBV

Commit message: finish schematic
Changed lines of the file:
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@@
-	)
-	(junction
-		(at 83.82 85.09)
-		(diameter 0)
-		(color 0 0 0 0)
 	)
 	(junction
@@
 	)
 	(junction
-		(at 133.35 82.55)
-		(diameter 0)
-		(color 0 0 0 0)
-	)
-	(junction
-		(at 133.35 85.09)
-		(diameter 0)
-		(color 0 0 0 0)
-	)
-	(junction
 		(at 52.07 77.47)
 		(diameter 0)
@@
 	(wire
 		(pts
-			(xy 133.35 82.55) (xy 123.19 82.55)
-		)
-		(stroke
-			(width 0)
-			(type default)
-		)
-	)
-	(wire
-		(pts
 			(xy 123.19 95.25) (xy 127 95.25)
 		)
@@
 	(wire
 		(pts
-			(xy 142.24 81.28) (xy 133.35 81.28)
-		)
-		(stroke
-			(width 0)
-			(type default)
-		)
-	)
-	(wire
-		(pts
 			(xy 145.415 100.33) (xy 153.67 100.33)
 		)
@@
 	(wire
 		(pts
-			(xy 86.36 86.36) (xy 83.82 86.36)
-		)
-		(stroke
-			(width 0)
-			(type default)
-		)
-	)
-	(wire
-		(pts
-			(xy 142.24 83.82) (xy 133.35 83.82)
-		)
-		(stroke
-			(width 0)
-			(type default)
-		)
-	)
-	(wire
-		(pts
 			(xy 148.59 65.405) (xy 148.59 67.945)
 		)
@@
 	(wire
 		(pts
-			(xy 133.35 81.28) (xy 133.35 82.55)
-		)
-		(stroke
-			(width 0)
-			(type default)
-		)
-	)
-	(wire
-		(pts
 			(xy 91.44 105.41) (xy 92.71 105.41)
 		)
@@
 	(wire
 		(pts
-			(xy 134.62 85.09) (xy 133.35 85.09)
+			(xy 134.62 85.09) (xy 123.19 85.09)
 		)
 		(stroke
@@
 	(wire
 		(pts
-			(xy 83.82 86.36) (xy 83.82 85.09)
-		)
-		(stroke
-			(width 0)
-			(type default)
-		)
-	)
-	(wire
-		(pts
 			(xy 207.01 143.51) (xy 207.01 146.05)
 		)
@@
 	(wire
 		(pts
-			(xy 134.62 82.55) (xy 133.35 82.55)
+			(xy 134.62 82.55) (xy 123.19 82.55)
 		)
 		(stroke
@@
 	(wire
 		(pts
-			(xy 133.35 85.09) (xy 123.19 85.09)
-		)
-		(stroke
-			(width 0)
-			(type default)
-		)
-	)
-	(wire
-		(pts
 			(xy 200.787 34.29) (xy 207.645 34.29)
 		)
@@
 	(wire
 		(pts
-			(xy 83.82 85.09) (xy 92.71 85.09)
-		)
-		(stroke
-			(width 0)
-			(type default)
-		)
-	)
-	(wire
-		(pts
 			(xy 148.59 57.785) (xy 148.59 55.245)
 		)
@@
 	(wire
 		(pts
-			(xy 81.915 85.09) (xy 83.82 85.09)
+			(xy 81.915 85.09) (xy 92.71 85.09)
 		)
 		(stroke
@@
 		(pts
 			(xy 67.945 170.815) (xy 75.565 170.815)
-		)
-		(stroke
-			(width 0)
-			(type default)
-		)
-	)
-	(wire
-		(pts
-			(xy 133.35 83.82) (xy 133.35 85.09)
 		)
 		(stroke
@@
 			)
 			(justify left bottom)
-		)
-	)
-	(global_label "RX"
-		(shape input)
-		(at 142.24 83.82 0)
-		(fields_autoplaced yes)
-		(effects
-			(font
-				(size 1.27 1.27)
-			)
-			(justify left)
-		)
-		(property "Intersheetrefs" "${INTERSHEET_REFS}"
-			(at 147.7047 83.82 0)
-			(hide yes)
-			(show_name no)
-			(do_not_autoplace no)
-			(effects
-				(font
-					(size 1.27 1.27)
-				)
-				(justify left)
-			)
 		)
 	)
@@
 			(hide yes)
 			(show_name no)
-			(do_not_autoplace no)
-			(effects
-				(font
-					(size 1.27 1.27)
-				)
-				(justify left)
-			)
-		)
-	)
-	(global_label "RST"
-		(shape input)
-		(at 86.36 86.36 0)
-		(fields_autoplaced yes)
-		(effects
-			(font
-				(size 1.27 1.27)
-			)
-			(justify left)
-		)
-		(property "Intersheetrefs" "${INTERSHEET_REFS}"
-			(at 92.7923 86.36 0)
-			(hide yes)
-			(show_name no)
-			(do_not_autoplace no)
-			(effects
-				(font
-					(size 1.27 1.27)
-				)
-				(justify left)
-			)
-		)
-	)
-	(global_label "TX"
-		(shape input)
-		(at 142.24 81.28 0)
-		(fields_autoplaced yes)
-		(effects
-			(font
-				(size 1.27 1.27)
-			)
-			(justify left)
-		)
-		(property "Intersheetrefs" "${INTERSHEET_REFS}"
-			(at 147.4023 81.28 0)
-			(hide yes)
-			(show_name no)
