File: kicad/_restore_backup_2026-08-13T12-33-19-172/bitcoinMiner.kicad_pcb (KiCad board)
At the start: 4 copper layers, 75 x 100 mm, 176 parts, among them J1 54-00164, J2 TC2030-IDC, J3 Conn_01x06, J4 USB_C_Receptacle_USB2.0_14P, J5 Conn_01x04, J6 Conn_01x04, J7 Conn_01x04_MountingPin, SW1 SW_Push, SW2 SW_Push, T1 net-tie, U10 ESP32-S3-WROOM-1, U11 EMC2101, U12 TPS546D24ARVFR, U2 25MHz, U3 TLV75712PDBV, U4 MCP1824T-0802E, U5 BM1370_mode1, U6 SN74LVC1T45DBV, U7 SN74LVC1T45DBV, U8 SN74LVC1T45DBV, U9 TLV75733PDBV

Commit message: add neopoixels and spinrender
Parts:
- removed C59, C60, C61, C62, C63, C64, C65, C66, C67: 0.1uF, Capacitor_SMD:C_0402_1005Metric
- removed D1, D2: LED, LED_SMD:LED_0603_1608Metric
- removed D10, D11, D3, D4, D5, D6, D7, D8, D9: WS2812B-2020, LED_SMD:LED_WS2812B-2020_PLCC4_2.0x2.0mm
- removed R24, R25: 10k, Resistor_SMD:R_0603_1608Metric
Connections:
- U10 pad 23: Net-(D2-A) -> /ESP32/GPIO21
- U10 pad 31: Net-(D3-DIN) -> /ESP32/GPIO38
Routing:
- net Net-(D3-DIN): track 93.2 -> 0.00 mm, vias 2 -> 0
- net Net-(D2-A): track 91.1 -> 0.00 mm, vias 2 -> 0
- net +5V: track 204.4 -> 122.4 mm, vias 73 -> 64
- net Net-(D4-DOUT): track 2.64 -> 0.00 mm
- net Net-(D7-DOUT): track 2.63 -> 0.00 mm
- net Net-(D6-DOUT): track 2.63 -> 0.00 mm
- net Net-(D3-DOUT): track 2.63 -> 0.00 mm
- net Net-(D10-DOUT): track 2.63 -> 0.00 mm
- net Net-(D10-DIN): track 2.63 -> 0.00 mm
- net Net-(D8-DOUT): track 2.63 -> 0.00 mm
- net Net-(D5-DOUT): track 2.61 -> 0.00 mm
- net Net-(D2-K): track 2.02 -> 0.00 mm
- net Net-(D1-K): track 2.02 -> 0.00 mm
- net GND: vias 148 -> 128
