File: kicad/bitcoinMiner.kicad_pcb (KiCad board)
At the start: 4 copper layers, 75 x 100 mm, 176 parts, among them J1 54-00164, J2 TC2030-IDC, J3 Conn_01x06, J4 USB_C_Receptacle_USB2.0_14P, J5 Conn_01x04, J6 Conn_01x04, J7 Conn_01x04_MountingPin, SW1 SW_Push, SW2 SW_Push, T1 net-tie, U10 ESP32-S3-WROOM-1, U11 EMC2101, U12 TPS546D24ARVFR, U2 25MHz, U3 TLV75712PDBV, U4 MCP1824T-0802E, U5 BM1370_mode1, U6 SN74LVC1T45DBV, U7 SN74LVC1T45DBV, U8 SN74LVC1T45DBV, U9 TLV75733PDBV

Commit message: add images and journal
Changed lines of the file:
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@@
 		)
 		(embedded_fonts no)
-		(model "${KICAD10_3DMODEL_DIR}/Connector_USB.3dshapes/USB_C_Receptacle_HRO_TYPE-C-31-M-12.step"
+		(model "${KICAD10_3DMODEL_DIR}/Connector_USB.3dshapes/USB_C_Receptacle_GCT_USB4105-xx-A_16P_TopMnt_Horizontal.step"
 			(offset
 				(xyz 0 0 0)
@@
 	)
 	(segment
-		(start 56 47)
-		(end 42 47)
+		(start 39.1 47.2)
+		(end 55.8 47.2)
 		(width 0.2)
 		(layer "F.Cu")
@@
 	)
 	(segment
-		(start 42 47)
-		(end 41.3 47.7)
+		(start 55.8 47.2)
+		(end 56 47)
 		(width 0.2)
 		(layer "F.Cu")
@@
 	)
 	(via
-		(at 41.3 47.7)
+		(at 39.1 47.2)
 		(size 0.6)
 		(drill 0.3)
@@
 	)
 	(segment
-		(start 41.3 47.7)
-		(end 40.7 47.7)
+		(start 39.1 47.2)
+		(end 39.1 46.1)
 		(width 0.2)
 		(layer "B.Cu")
@@
 	)
 	(segment
-		(start 40.7 47.7)
+		(start 39.1 46.1)
 		(end 25 32)
 		(width 0.2)
